File: TSOC_CYBLE/revisions/R1_0/TSOC_CYBLE_R1_0.brd (EAGLE design)
At the start: 44.5 x 30.5 mm, 46 parts, among them J2 JTAG-ISSPMIN, Q1 FDG1024NZ, Q2 FDC6420C, U1 MIC5219 3.3V, U2 CYBLE-022001-00

Commit message: update images
Parts:
- added D2: 20V-1A, Seeed-Diode-2016:SOD-123
Connections:
- new net VIN: C1.2, D1.-, D2.-, U1.1, U1.3
- net 5V0: now also D2.+; no longer C1.2, D1.-, U1.1, U1.3
Routing:
- net 5V0: track 15.5 -> 1.90 mm
- net VIN: track 0.00 -> 10.3 mm
Changed lines of the file:
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@@
 <layer number="220" name="220bmp" color="21" fill="1" visible="no" active="no"/>
 <layer number="221" name="221bmp" color="22" fill="1" visible="no" active="no"/>
+<layer number="222" name="222bmp" color="23" fill="1" visible="no" active="no"/>
 <layer number="223" name="223bmp" color="24" fill="1" visible="no" active="no"/>
 <layer number="224" name="224bmp" color="25" fill="1" visible="no" active="no"/>
@@
 <attribute name="VALUE" x="10.4775" y="16.5735" size="0.4064" layer="27"/>
 </element>
+<element name="D2" library="Seeed-Diode-2016" package="SOD-123" value="20V-1A" x="11.938" y="7.366" smashed="yes" rot="R90">
+<attribute name="MPN" value="B5819W" x="18.796" y="4.064" size="1.778" layer="27" rot="R90" display="off"/>
+<attribute name="NAME" x="10.541" y="6.731" size="0.889" layer="25" font="vector" ratio="15" rot="R90"/>
+<attribute name="VALUE" x="13.97" y="5.461" size="0.889" layer="27" font="vector" ratio="11" rot="R90"/>
+<attribute name="NAME" x="12.573" y="6.477" size="0.381" layer="33" ratio="10" rot="R90"/>
+</element>
 <element name="D1" library="Seeed-Diode-2016" package="SOD-123" value="20V-1A" x="10.541" y="10.795" smashed="yes">
 <attribute name="MPN" value="B5819W" x="7.239" y="3.937" size="1.778" layer="27" display="off"/>
@@
 <wire x1="9.4234" y1="26.1366" x2="9.398" y2="26.67" width="0.1778" layer="16"/>
 <wire x1="9.779" y1="27.7368" x2="9.860921875" y2="27.787596875" width="0.1778" layer="16"/>
-<wire x1="23.4696" y1="27.0256" x2="23.4442" y2="27.0256" width="0.1778" layer="16"/>
-<wire x1="26.8478" y1="24.1808" x2="26.8478" y2="24.13" width="0.1778" layer="16"/>
-<wire x1="9.2456" y1="26.3144" x2="9.398" y2="26.67" width="0.1778" layer="16"/>
-<wire x1="9.2456" y1="26.3144" x2="9.271" y2="26.3144" width="0.1778" layer="16"/>
 </signal>
 <signal name="RXD">
@@
 <signal name="5V0">
 <contactref element="TSOC" pad="11C"/>
-<contactref element="U1" pad="1"/>
-<contactref element="U1" pad="3"/>
-<contactref element="D1" pad="-"/>
-<contactref element="C1" pad="2"/>
-<wire x1="12.38" y1="15.4639" x2="12.38" y2="13.269" width="0.6096" layer="1"/>
-<wire x1="12.38" y1="13.269" x2="12.319" y2="13.208" width="0.6096" layer="1"/>
-<wire x1="10.48" y1="15.4639" x2="10.48" y2="13.904" width="0.6096" layer="1"/>
-<wire x1="10.48" y1="13.904" x2="10.922" y2="13.462" width="0.6096" layer="1"/>
-<wire x1="10.922" y1="13.462" x2="12.065" y2="13.462" width="0.6096" layer="1"/>
-<wire x1="12.065" y1="13.462" x2="12.319" y2="13.208" width="0.6096" layer="1"/>
-<wire x1="12.192" y1="10.795" x2="12.192" y2="13.081" width="0.8128" layer="1"/>
-<wire x1="12.192" y1="13.081" x2="12.319" y2="13.208" width="0.8128" layer="1"/>
-<wire x1="11.938" y1="3.81" x2="11.938" y2="10.541" width="0.8128" layer="1"/>
-<wire x1="11.938" y1="10.541" x2="12.192" y2="10.795" width="0.8128" layer="1"/>
+<contactref element="D2" pad="+"/>
+<wire x1="11.938" y1="5.715" x2="11.938" y2="3.81" width="0.8128" layer="1"/>
 </signal>
 <signal name="A0">
@@
 <wire x1="12.446" y1="18.796" x2="13.843" y2="18.796" width="0.6096" layer="1"/>
 </signal>
+<signal name="VIN">
+<contactref element="U1" pad="1"/>
+<contactref element="U1" pad="3"/>
+<contactref element="D2" pad="-"/>
+<contactref element="D1" pad="-"/>
+<contactref element="C1" pad="2"/>
+<wire x1="12.38" y1="15.4639" x2="12.38" y2="13.269" width="0.6096" layer="1"/>
+<wire x1="12.38" y1="13.269" x2="12.319" y2="13.208" width="0.6096" layer="1"/>
+<wire x1="10.48" y1="15.4639" x2="10.48" y2="13.904" width="0.6096" layer="1"/>
+<wire x1="10.48" y1="13.904" x2="10.922" y2="13.462" width="0.6096" layer="1"/>
+<wire x1="10.922" y1="13.462" x2="12.065" y2="13.462" width="0.6096" layer="1"/>
+<wire x1="12.065" y1="13.462" x2="12.319" y2="13.208" width="0.6096" layer="1"/>
+<wire x1="11.938" y1="9.017" x2="11.938" y2="10.541" width="0.8128" layer="1"/>
+<wire x1="11.938" y1="10.541" x2="12.192" y2="10.795" width="0.8128" layer="1"/>
+<wire x1="12.192" y1="10.795" x2="12.192" y2="13.081" width="0.8128" layer="1"/>
+<wire x1="12.192" y1="13.081" x2="12.319" y2="13.208" width="0.8128" layer="1"/>
+</signal>
 <signal name="VDDR">
