File: TSOC_CYBLE/revisions/R1_0/TSOC_CYBLE_R1_0.sch (EAGLE design)
At the start: 45 parts, among them J2 JTAG-ISSPMIN, Q1 FDG1024NZ, Q2 FDC6420C, U1 MIC5219 3.3V, U2 CYBLE-022001-00

Commit message: update images
Parts:
- added D2: 20V-1A, Seeed-Diode-2016:SMD-DIODE-SCHOTTKY-20V-1A(SOD-123)
Connections:
- new net VIN: C1.2, D1.-, D2.-, U1.EN, U1.IN
- net 5V0: now also D2.+; no longer C1.2, D1.-, U1.EN, U1.IN
Changed lines of the file:
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@@
 <part name="GND12" library="SparkFun" deviceset="GND" device=""/>
 <part name="U$16" library="PatternAgents-Beautify" deviceset="GND" device=""/>
+<part name="D2" library="Seeed-Diode-2016" deviceset="SMD-DIODE-SCHOTTKY-20V-1A(SOD-123)" device="" value="20V-1A"/>
 <part name="D1" library="Seeed-Diode-2016" deviceset="SMD-DIODE-SCHOTTKY-20V-1A(SOD-123)" device="" value="20V-1A"/>
 <part name="BOOT" library="TSOC_GROVEY_WIFI" deviceset="SMD-BUTTON-TOP-DHT-4235A(4P-4.2X3.2MM)" device="" value="DHT-4235A"/>
@@
 <instance part="GND12" gate="1" x="406.4" y="96.52"/>
 <instance part="U$16" gate="G$1" x="398.78" y="99.06"/>
+<instance part="D2" gate="G$1" x="386.08" y="127"/>
 <instance part="D1" gate="G$1" x="386.08" y="116.84"/>
 <instance part="BOOT" gate="G$1" x="55.88" y="327.66"/>
@@
 </segment>
 <segment>
-<pinref part="U1" gate="G$1" pin="IN"/>
-<wire x1="414.02" y1="124.46" x2="398.78" y2="124.46" width="0.1524" layer="91"/>
-<wire x1="398.78" y1="111.76" x2="398.78" y2="116.84" width="0.1524" layer="91"/>
-<wire x1="398.78" y1="116.84" x2="398.78" y2="119.38" width="0.1524" layer="91"/>
-<wire x1="398.78" y1="119.38" x2="398.78" y2="124.46" width="0.1524" layer="91"/>
-<junction x="398.78" y="124.46"/>
-<junction x="398.78" y="119.38"/>
-<pinref part="U1" gate="G$1" pin="EN"/>
-<wire x1="398.78" y1="119.38" x2="414.02" y2="119.38" width="0.1524" layer="91"/>
-<wire x1="398.78" y1="124.46" x2="398.78" y2="139.7" width="0.1524" layer="91"/>
-<wire x1="398.78" y1="139.7" x2="472.44" y2="139.7" width="0.1524" layer="91"/>
-<label x="472.44" y="139.7" size="1.27" layer="95" ratio="10" xref="yes"/>
-<junction x="398.78" y="116.84"/>
-<wire x1="389.89" y1="116.84" x2="398.78" y2="116.84" width="0.1524" layer="91"/>
-<pinref part="D1" gate="G$1" pin="-"/>
-<pinref part="C1" gate="G$1" pin="2"/>
+<label x="373.38" y="127" size="1.27" layer="95" ratio="10" rot="R180" xref="yes"/>
+<pinref part="D2" gate="G$1" pin="+"/>
+<wire x1="382.27" y1="127" x2="373.38" y2="127" width="0.1524" layer="91"/>
 </segment>
 </net>
@@
 </segment>
 </net>
+<net name="VIN" class="0">
+<segment>
+<pinref part="U1" gate="G$1" pin="IN"/>
+<wire x1="414.02" y1="124.46" x2="398.78" y2="124.46" width="0.1524" layer="91"/>
+<wire x1="398.78" y1="111.76" x2="398.78" y2="116.84" width="0.1524" layer="91"/>
+<wire x1="398.78" y1="116.84" x2="398.78" y2="119.38" width="0.1524" layer="91"/>
+<wire x1="398.78" y1="119.38" x2="398.78" y2="124.46" width="0.1524" layer="91"/>
+<junction x="398.78" y="124.46"/>
+<junction x="398.78" y="119.38"/>
+<pinref part="U1" gate="G$1" pin="EN"/>
+<wire x1="398.78" y1="119.38" x2="414.02" y2="119.38" width="0.1524" layer="91"/>
+<wire x1="398.78" y1="124.46" x2="398.78" y2="127" width="0.1524" layer="91"/>
+<wire x1="398.78" y1="127" x2="398.78" y2="139.7" width="0.1524" layer="91"/>
+<wire x1="398.78" y1="139.7" x2="472.44" y2="139.7" width="0.1524" layer="91"/>
+<label x="472.44" y="139.7" size="1.27" layer="95" ratio="10" xref="yes"/>
+<junction x="398.78" y="116.84"/>
+<wire x1="389.89" y1="116.84" x2="398.78" y2="116.84" width="0.1524" layer="91"/>
+<junction x="398.78" y="127"/>
+<pinref part="D2" gate="G$1" pin="-"/>
+<wire x1="389.89" y1="127" x2="398.78" y2="127" width="0.1524" layer="91"/>
+<pinref part="D1" gate="G$1" pin="-"/>
+<pinref part="C1" gate="G$1" pin="2"/>
+</segment>
+</net>
